File: board_carrier/board_carrier.sch (KiCad schematic (older format))
At the start: 13 parts, among them J1 Conn_01x08, J2 Conn_01x08, J3 Conn_01x04, U1 TJA1051T-3, U2 LM78M05_TO252

Commit message: carrier with mx120
Parts:
- removed J3: Conn_01x04, Connector_Molex:Molex_Micro-Fit_3.0_43650-0415_1x04_P3.00mm_Vertical, symbol Connector_Generic:Conn_01x04
- removed J_LSU1: Conn_01x06, Connector_Molex:Molex_Micro-Fit_3.0_43650-0615_1x06_P3.00mm_Vertical, symbol Connector_Generic:Conn_01x06
- added J3: Conn_02x06_Top_Bottom, mx120:mx120g-12, symbol Connector_Generic:Conn_02x06_Top_Bottom
Connections:
- net 12V_RAW: now also J3.6 (Pin_6)
- net CAN_H: now also J3.11 (Pin_11)
- net CAN_L: now also J3.12 (Pin_12)
- net GND: now also J3.1 (Pin_1)
- net LSU_Heater+: now also J3.4 (Pin_4)
- net LSU_Heater-: now also J3.3 (Pin_3)
- net LSU_Ip: now also J3.2 (Pin_2)
- net LSU_Rtrim: now also J3.8 (Pin_8)
- net LSU_Un: now also J3.9 (Pin_9)
- net LSU_Vm: now also J3.7 (Pin_7)
- no-connect marks 0 -> 1
Changed lines of the file:
@@
 Text Label 2700 2450 2    50   ~ 0
 LSU_Heater-
-Text Label 4100 3200 2    50   ~ 0
+Text Label 925  4250 0    50   ~ 0
 LSU_Heater-
-Text Label 4100 3000 2    50   ~ 0
+Text Label 925  4150 0    50   ~ 0
 LSU_Ip
-Text Label 4100 3100 2    50   ~ 0
+Text Label 2525 4050 2    50   ~ 0
 LSU_Vm
-Text Label 4100 3400 2    50   ~ 0
+Text Label 2525 4150 2    50   ~ 0
 LSU_Rtrim
-Text Label 4100 3500 2    50   ~ 0
+Text Label 2525 4250 2    50   ~ 0
 LSU_Un
 Text Label 1825 675  0    50   ~ 0
@@
 Wire Wire Line
 	1825 675  1825 1075
-Text Label 4100 3300 2    50   ~ 0
+Text Label 925  4350 0    50   ~ 0
 LSU_Heater+
-$Comp
-L Connector_Generic:Conn_01x06 J_LSU1
-U 1 1 5FBB3B15
-P 3350 3200
-F 0 "J_LSU1" H 3268 3525 50  0000 C CNN
-F 1 "Conn_01x06" H 3268 2766 50  0001 C CNN
-F 2 "Connector_Molex:Molex_Micro-Fit_3.0_43650-0615_1x06_P3.00mm_Vertical" H 3350 3200 50  0001 C CNN
-F 3 "~" H 3350 3200 50  0001 C CNN
-	1    3350 3200
-	-1   0    0    -1
-$EndComp
 Wire Wire Line
-	3550 3300 4100 3300
+	1475 4350 925  4350
 Wire Wire Line
-	4100 3200 3550 3200
+	925  4250 1475 4250
 Wire Wire Line
-	4100 3000 3550 3000
+	925  4150 1475 4150
 Wire Wire Line
-	3550 3100 4100 3100
+	1975 4050 2525 4050
 Wire Wire Line
-	3550 3400 4100 3400
+	1975 4150 2525 4150
 Wire Wire Line
-	3550 3500 4100 3500
-Text Notes 4175 3000 0    50   ~ 0
+	1975 4250 2525 4250
+Text Notes 850  4150 2    50   ~ 0
 red
-Text Notes 4175 3100 0    50   ~ 0
+Text Notes 2600 4050 0    50   ~ 0
 yellow
-Text Notes 4175 3200 0    50   ~ 0
+Text Notes 850  4300 2    50   ~ 0
 white
-Text Notes 4175 3300 0    50   ~ 0
+Text Notes 850  4400 2    50   ~ 0
 grey
-Text Notes 4175 3400 0    50   ~ 0
+Text Notes 2600 4150 0    50   ~ 0
 green
-Text Notes 4175 3500 0    50   ~ 0
+Text Notes 2600 4250 0    50   ~ 0
 black
 Text Notes 4175 2875 0    50   ~ 0
 LSU 4.9 Wire Colors:
 $Comp
-L Connector_Generic:Conn_01x04 J3
-U 1 1 5FBCCED0
-P 1325 3800
-F 0 "J3" H 1243 4025 50  0000 C CNN
-F 1 "Conn_01x04" H 1243 4026 50  0001 C CNN
-F 2 "Connector_Molex:Molex_Micro-Fit_3.0_43650-0415_1x04_P3.00mm_Vertical" H 1325 3800 50  0001 C CNN
-F 3 "~" H 1325 3800 50  0001 C CNN
-	1    1325 3800
-	-1   0    0    -1
-$EndComp
-$Comp
 L power:GND #PWR0114
 U 1 1 5FBCD9A4
-P 1600 4100
-F 0 "#PWR0114" H 1600 3850 50  0001 C CNN
-F 1 "GND" V 1605 3972 50  0000 R CNN
-F 2 "" H 1600 4100 50  0001 C CNN
-F 3 "" H 1600 4100 50  0001 C CNN
-	1    1600 4100
+P 5475 4925
+F 0 "#PWR0114" H 5475 4675 50  0001 C CNN
+F 1 "GND" V 5480 4797 50  0000 R CNN
+F 2 "" H 5475 4925 50  0001 C CNN
+F 3 "" H 5475 4925 50  0001 C CNN
+	1    5475 4925
 	1    0    0    -1
 $EndComp
 Wire Wire Line
-	1525 4000 1600 4000
+	5400 4825 5475 4825
 Wire Wire Line
-	1600 4000 1600 4100
-Text GLabel 1650 3625 2    50   Input ~ 0
+	5475 4825 5475 4925
+Text GLabel 1400 4550 0    50   Input ~ 0
 12V_RAW
 Wire Wire Line
-	1650 3625 1525 3700
-Text Label 1825 3800 2    50   ~ 0
+	1400 4550 1475 4550
+Text Label 2275 4450 2    50   ~ 0
 CAN_H
-Text Label 1825 3900 2    50   ~ 0
+Text Label 2275 4550 2    50   ~ 0
 CAN_L
 Wire Wire Line
-	1825 3900 1525 3900
+	2275 4550 1975 4550
 Wire Wire Line
-	1825 3800 1525 3800
+	2275 4450 1975 4450
+$Comp
+L Connector_Generic:Conn_02x06_Top_Bottom J3
+U 1 1 5FD3D185
+P 1675 4250
+F 0 "J3" H 1725 4667 50  0000 C CNN
+F 1 "Conn_02x06_Top_Bottom" H 1725 4576 50  0000 C CNN
+F 2 "mx120:mx120g-12" H 1675 4250 50  0001 C CNN
+F 3 "~" H 1675 4250 50  0001 C CNN
+	1    1675 4250
+	1    0    0    -1
+$EndComp
+$Comp
+L power:GND #PWR0115
+U 1 1 5FD4C273
+P 1350 4050
+F 0 "#PWR0115" H 1350 3800 50  0001 C CNN
+F 1 "GND" V 1355 3922 50  0000 R CNN
+F 2 "" H 1350 4050 50  0001 C CNN
+F 3 "" H 1350 4050 50  0001 C CNN
+	1    1350 4050
+	0    1    1    0
+$EndComp
+Wire Wire Line
+	1350 4050 1475 4050
+NoConn ~ 1475 4450
 $EndSCHEMATC

Commit message: minor
Connections:
- no-connect marks 1 -> 2
Changed lines of the file:
@@
 	1350 4050 1475 4050
 NoConn ~ 1475 4450
+NoConn ~ 1975 4350
 $EndSCHEMATC

Commit message: carrier mods
Connections:
- net LSU_Rtrim: now also J3.9 (Pin_9); no longer J3.8 (Pin_8)
- net LSU_Un: now also J3.10 (Pin_10); no longer J3.9 (Pin_9)
- net LSU_Vm: now also J3.8 (Pin_8); no longer J3.7 (Pin_7)
Other:
- note removed: "LSU 4.9 Wire Colors:"
- moved on the sheet: J3, U1
Changed lines of the file:
@@
 L power:GND #PWR0101
 U 1 1 5FB6223C
-P 5475 1800
-F 0 "#PWR0101" H 5475 1550 50  0001 C CNN
-F 1 "GND" H 5480 1627 50  0000 C CNN
-F 2 "" H 5475 1800 50  0001 C CNN
-F 3 "" H 5475 1800 50  0001 C CNN
-	1    5475 1800
+P 5075 1800
+F 0 "#PWR0101" H 5075 1550 50  0001 C CNN
+F 1 "GND" H 5080 1627 50  0000 C CNN
+F 2 "" H 5075 1800 50  0001 C CNN
+F 3 "" H 5075 1800 50  0001 C CNN
+	1    5075 1800
 	1    0    0    -1
 $EndComp
@@
 L Interface_CAN_LIN:TJA1051T-3 U1
 U 1 1 5FB6A2CB
-P 5475 1400
-F 0 "U1" H 5150 1775 50  0000 C CNN
-F 1 "TJA1051T-3" H 5750 1775 50  0000 C CNN
-F 2 "Package_SO:SOIC-8_3.9x4.9mm_P1.27mm" H 5475 900 50  0001 C CIN
-F 3 "http://www.nxp.com/documents/data_sheet/TJA1051.pdf" H 5475 1400 50  0001 C CNN
-F 4 "C38695" H 5475 1400 50  0001 C CNN "LCSC"
-	1    5475 1400
+P 5075 1400
+F 0 "U1" H 4750 1775 50  0000 C CNN
+F 1 "TJA1051T-3" H 5350 1775 50  0000 C CNN
+F 2 "Package_SO:SOIC-8_3.9x4.9mm_P1.27mm" H 5075 900 50  0001 C CIN
+F 3 "http://www.nxp.com/documents/data_sheet/TJA1051.pdf" H 5075 1400 50  0001 C CNN
+F 4 "C38695" H 5075 1400 50  0001 C CNN "LCSC"
+	1    5075 1400
 	1    0    0    -1
 $EndComp
@@
 L power:+5V #PWR0106
 U 1 1 5FB6B936
-P 5475 1000
-F 0 "#PWR0106" H 5475 850 50  0001 C CNN
-F 1 "+5V" H 5490 1173 50  0000 C CNN
-F 2 "" H 5475 1000 50  0001 C CNN
-F 3 "" H 5475 1000 50  0001 C CNN
-	1    5475 1000
+P 5075 1000
+F 0 "#PWR0106" H 5075 850 50  0001 C CNN
+F 1 "+5V" H 5090 1173 50  0000 C CNN
+F 2 "" H 5075 1000 50  0001 C CNN
+F 3 "" H 5075 1000 50  0001 C CNN
+	1    5075 1000
 	1    0    0    -1
 $EndComp
@@
 L power:GND #PWR0107
 U 1 1 5FB6BFE5
-P 4975 1600
-F 0 "#PWR0107" H 4975 1350 50  0001 C CNN
-F 1 "GND" V 4980 1472 50  0000 R CNN
-F 2 "" H 4975 1600 50  0001 C CNN
-F 3 "" H 4975 1600 50  0001 C CNN
-	1    4975 1600
+P 4575 1600
+F 0 "#PWR0107" H 4575 1350 50  0001 C CNN
+F 1 "GND" V 4580 1472 50  0000 R CNN
+F 2 "" H 4575 1600 50  0001 C CNN
+F 3 "" H 4575 1600 50  0001 C CNN
+	1    4575 1600
 	0    1    1    0
 $EndComp
@@
 	1    0    0    -1
 $EndComp
-Text Label 4650 1200 0    50   ~ 0
+Text Label 4250 1200 0    50   ~ 0
 CAN_TX
 Wire Wire Line
-	4650 1200 4975 1200
-Wire Wire Line
-	4975 1300 4650 1300
-Text Label 4650 1300 0    50   ~ 0
+	4250 1200 4575 1200
+Wire Wire Line
+	4575 1300 4250 1300
+Text Label 4250 1300 0    50   ~ 0
 CAN_RX
-Text Label 6275 1300 2    50   ~ 0
+Text Label 5875 1300 2    50   ~ 0
 CAN_H
-Text Label 6275 1500 2    50   ~ 0
+Text Label 5875 1500 2    50   ~ 0
 CAN_L
 Wire Wire Line
-	6275 1500 5975 1500
-Wire Wire Line
-	6275 1300 5975 1300
+	5875 1500 5575 1500
+Wire Wire Line
+	5875 1300 5575 1300
 $Comp
 L Device:R R1
@@
 Connection ~ 3800 1500
 Wire Wire Line
-	3800 1500 4975 1500
+	3800 1500 4575 1500
 Text Notes 3350 2350 0    50   ~ 0
 VIO pin only draws 500uA max so\na divider will work fine
@@
 Text Label 2700 2450 2    50   ~ 0
 LSU_Heater-
-Text Label 925  4250 0    50   ~ 0
+Text Label 1525 3900 0    50   ~ 0
 LSU_Heater-
-Text Label 925  4150 0    50   ~ 0
+Text Label 1525 3800 0    50   ~ 0
 LSU_Ip
-Text Label 2525 4050 2    50   ~ 0
-LSU_Vm
-Text Label 2525 4150 2    50   ~ 0
-LSU_Rtrim
-Text Label 2525 4250 2    50   ~ 0
-LSU_Un
 Text Label 1825 675  0    50   ~ 0
 LSU_Heater+
 Wire Wire Line
 	1825 675  1825 1075
-Text Label 925  4350 0    50   ~ 0
+Text Label 1525 4000 0    50   ~ 0
 LSU_Heater+
 Wire Wire Line
-	1475 4350 925  4350
-Wire Wire Line
-	925  4250 1475 4250
-Wire Wire Line
-	925  4150 1475 4150
-Wire Wire Line
-	1975 4050 2525 4050
-Wire Wire Line
-	1975 4150 2525 4150
-Wire Wire Line
-	1975 4250 2525 4250
-Text Notes 850  4150 2    50   ~ 0
+	2075 4000 1525 4000
+Wire Wire Line
+	1525 3900 2075 3900
+Wire Wire Line
+	1525 3800 2075 3800
+Text Notes 1450 3800 2    50   ~ 0
 red
-Text Notes 2600 4050 0    50   ~ 0
-yellow
-Text Notes 850  4300 2    50   ~ 0
+Text Notes 1450 3950 2    50   ~ 0
 white
-Text Notes 850  4400 2    50   ~ 0
+Text Notes 1450 4050 2    50   ~ 0
 grey
-Text Notes 2600 4150 0    50   ~ 0
-green
-Text Notes 2600 4250 0    50   ~ 0
-black
-Text Notes 4175 2875 0    50   ~ 0
-LSU 4.9 Wire Colors:
-$Comp
-L power:GND #PWR0114
-U 1 1 5FBCD9A4
-P 5475 4925
-F 0 "#PWR0114" H 5475 4675 50  0001 C CNN
-F 1 "GND" V 5480 4797 50  0000 R CNN
-F 2 "" H 5475 4925 50  0001 C CNN
-F 3 "" H 5475 4925 50  0001 C CNN
-	1    5475 4925
-	1    0    0    -1
-$EndComp
-Wire Wire Line
-	5400 4825 5475 4825
-Wire Wire Line
-	5475 4825 5475 4925
-Text GLabel 1400 4550 0    50   Input ~ 0
+Text GLabel 2000 4200 0    50   Input ~ 0
 12V_RAW
 Wire Wire Line
-	1400 4550 1475 4550
-Text Label 2275 4450 2    50   ~ 0
+	2000 4200 2075 4200
+Text Label 2875 4100 2    50   ~ 0
 CAN_H
-Text Label 2275 4550 2    50   ~ 0
+Text Label 2875 4200 2    50   ~ 0
 CAN_L
 Wire Wire Line
-	2275 4550 1975 4550
-Wire Wire Line
-	2275 4450 1975 4450
+	2875 4200 2575 4200
+Wire Wire Line
+	2875 4100 2575 4100
 $Comp
 L Connector_Generic:Conn_02x06_Top_Bottom J3
 U 1 1 5FD3D185
-P 1675 4250
-F 0 "J3" H 1725 4667 50  0000 C CNN
-F 1 "Conn_02x06_Top_Bottom" H 1725 4576 50  0000 C CNN
-F 2 "mx120:mx120g-12" H 1675 4250 50  0001 C CNN
-F 3 "~" H 1675 4250 50  0001 C CNN
-	1    1675 4250
+P 2275 3900
+F 0 "J3" H 2325 4317 50  0000 C CNN
+F 1 "Conn_02x06_Top_Bottom" H 2325 4226 50  0000 C CNN
+F 2 "mx120:mx120g-12" H 2275 3900 50  0001 C CNN
+F 3 "~" H 2275 3900 50  0001 C CNN
+	1    2275 3900
 	1    0    0    -1
 $EndComp
@@
 L power:GND #PWR0115
 U 1 1 5FD4C273
-P 1350 4050
-F 0 "#PWR0115" H 1350 3800 50  0001 C CNN
-F 1 "GND" V 1355 3922 50  0000 R CNN
-F 2 "" H 1350 4050 50  0001 C CNN
-F 3 "" H 1350 4050 50  0001 C CNN
-	1    1350 4050
+P 1950 3700
+F 0 "#PWR0115" H 1950 3450 50  0001 C CNN
+F 1 "GND" V 1955 3572 50  0000 R CNN
+F 2 "" H 1950 3700 50  0001 C CNN
+F 3 "" H 1950 3700 50  0001 C CNN
+	1    1950 3700
 	0    1    1    0
 $EndComp
 Wire Wire Line
-	1350 4050 1475 4050
-NoConn ~ 1475 4450
-NoConn ~ 1975 4350
+	1950 3700 2075 3700
+NoConn ~ 2075 4100
+Text Notes 3200 4000 0    50   ~ 0
+black
+Text Notes 3200 3900 0    50   ~ 0
+green
+Text Notes 3200 3800 0    50   ~ 0
+yellow
+Wire Wire Line
+	2575 4000 3125 4000
+Wire Wire Line
+	2575 3900 3125 3900
+Wire Wire Line
+	2575 3800 3125 3800
+Text Label 3125 4000 2    50   ~ 0
+LSU_Un
+Text Label 3125 3900 2    50   ~ 0
+LSU_Rtrim
+Text Label 3125 3800 2    50   ~ 0
+LSU_Vm
+NoConn ~ 2575 3700
 $EndSCHEMATC
