File: board_carrier/board_carrier.sch (KiCad schematic (older format))
At the start: 12 parts, among them J1 Conn_01x08, J2 Conn_01x08, J3 Conn_02x06_Top_Bottom, U1 TJA1051T-3, U2 LM78M05_TO252

Commit message: add CAN caps, solid reg pad
Parts:
- added C4, C5: 47p, Capacitor_SMD:C_0402_1005Metric, symbol Device:C
Connections:
- net CAN_H: now also C4.2
- net CAN_L: now also C5.1
- net GND: now also C4.1, C5.2
Changed lines of the file:
@@
 P 7325 3725
 F 0 "#PWR0101" H 7325 3475 50  0001 C CNN
-F 1 "GND" H 7330 3552 50  0000 C CNN
+F 1 "GND" H 7330 3552 50  0001 C CNN
 F 2 "" H 7325 3725 50  0001 C CNN
 F 3 "" H 7325 3725 50  0001 C CNN
@@
 Text Label 6500 3225 0    50   ~ 0
 CAN_RX
-Text Label 8125 3225 2    50   ~ 0
+Text Label 8400 3225 2    50   ~ 0
 CAN_H
-Text Label 8125 3425 2    50   ~ 0
+Text Label 8400 3425 2    50   ~ 0
 CAN_L
 Wire Wire Line
-	8125 3425 7825 3425
-Wire Wire Line
-	8125 3225 7825 3225
+	8400 3425 8050 3425
+Wire Wire Line
+	8400 3225 8050 3225
 $Comp
 L Device:R R1
@@
 LSU_Vm
 NoConn ~ 4825 5625
+$Comp
+L Device:C C4
+U 1 1 5FC74FFA
+P 8050 2975
+F 0 "C4" H 8165 3021 50  0000 L CNN
+F 1 "47p" H 8165 2930 50  0000 L CNN
+F 2 "Capacitor_SMD:C_0402_1005Metric" H 8088 2825 50  0001 C CNN
+F 3 "~" H 8050 2975 50  0001 C CNN
+F 4 "C1567" H 8050 2975 50  0001 C CNN "LCSC"
+	1    8050 2975
+	1    0    0    -1
+$EndComp
+$Comp
+L Device:C C5
+U 1 1 5FC7558C
+P 8050 3675
+F 0 "C5" H 8165 3721 50  0000 L CNN
+F 1 "47p" H 8165 3630 50  0000 L CNN
+F 2 "Capacitor_SMD:C_0402_1005Metric" H 8088 3525 50  0001 C CNN
+F 3 "~" H 8050 3675 50  0001 C CNN
+F 4 "C1567" H 8050 3675 50  0001 C CNN "LCSC"
+	1    8050 3675
+	1    0    0    -1
+$EndComp
+$Comp
+L power:GND #PWR0114
+U 1 1 5FC75D4C
+P 8050 3825
+F 0 "#PWR0114" H 8050 3575 50  0001 C CNN
+F 1 "GND" H 8055 3652 50  0001 C CNN
+F 2 "" H 8050 3825 50  0001 C CNN
+F 3 "" H 8050 3825 50  0001 C CNN
+	1    8050 3825
+	1    0    0    -1
+$EndComp
+$Comp
+L power:GND #PWR0116
+U 1 1 5FC761A0
+P 8050 2825
+F 0 "#PWR0116" H 8050 2575 50  0001 C CNN
+F 1 "GND" H 8055 2652 50  0001 C CNN
+F 2 "" H 8050 2825 50  0001 C CNN
+F 3 "" H 8050 2825 50  0001 C CNN
+	1    8050 2825
+	-1   0    0    1
+$EndComp
+Wire Wire Line
+	8050 3125 8050 3225
+Connection ~ 8050 3225
+Wire Wire Line
+	8050 3225 7825 3225
+Wire Wire Line
+	8050 3425 8050 3525
+Connection ~ 8050 3425
+Wire Wire Line
+	8050 3425 7825 3425
 $EndSCHEMATC

Commit message: moar caps
Parts:
- added C10, C7, C8, C9: 10u, Capacitor_SMD:C_1206_3216Metric, symbol Device:C
- added C6: 22u, Capacitor_SMD:C_0805_2012Metric, symbol Device:C
Connections:
- net +5V: now also C6.1
- net 12V_RAW: now also C7.1, C8.2, C9.1
- net GND: now also C10.2, C6.2, C7.2, C8.1, C9.2
- net LSU_Heater+: now also C10.1
Other:
- moved on the sheet: C1, C2, D1, D2, U2

Commit message: switch to better diode
Parts:
- D2: LCSC C8678 -> C22452
Changed lines of the file:
@@
 F 2 "Diode_SMD:D_SMA" H 3050 3000 50  0001 C CNN
 F 3 "~" H 3050 3000 50  0001 C CNN
-F 4 "C8678" H 3050 3000 50  0001 C CNN "LCSC"
+F 4 "C22452" H 3050 3000 50  0001 C CNN "LCSC"
 	1    3050 3000
 	-1   0    0    1

Commit message: lower voltage tvs
Parts:
- D1: LCSC C133648 -> C151279
Changed lines of the file:
@@
 F 2 "Diode_SMD:D_SMC" H 1500 3275 50  0001 C CNN
 F 3 "~" H 1500 3275 50  0001 C CNN
-F 4 "C133648" H 1500 3275 50  0001 C CNN "LCSC"
+F 4 "C151279" H 1500 3275 50  0001 C CNN "LCSC"
 	1    1500 3275
 	0    1    1    0
