File: hardware/board_module/wideband_controller.kicad_sch (KiCad schematic)
At the start: 57 parts, among them J1 Conn_01x08, J2 Conn_ARM_SWD_TagConnect_TC2030, J3 Conn_01x08, Q1 BTS3028, U1 MCP6004, U2 STM32F042K6Tx, U3 REF3033, U5 AD8628, U9 XC6206P332MR

Commit message: vbatt sense
Parts:
- added C6: 1u, Capacitor_SMD:C_0402_1005Metric, symbol Device:C
- added R20: 100k, Resistor_SMD:R_0402_1005Metric, symbol Device:R
- added R21: 10k, Resistor_SMD:R_0402_1005Metric, symbol Device:R
Connections:
- net GND: now also C6.2, R21.2
- net nRESET: no longer J3.7 (Pin_7)
- net at U2.14 (PB0): now also C6.1, R20.2, R21.1
- new net VBatt_Sense: J3.7 (Pin_7), R20.1
- no-connect marks 9 -> 8
Other:
- moved on the sheet: C16, R29, U2

Commit message: update kicad & bom tweaks
Parts:
- J1, J3: LCSC (none) -> C32713274
- Q1: value BTS3028 -> VND14NV04; LCSC C112639 -> C2649436

Commit message: rev C: just BOM improvements
Other:
- company: (none) -> FOME / Happy Cactus Garage
- title: (none) -> FOME Open Source Wideband O2 Module
Changed lines of the file:
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@@
 	(generator_version "9.0")
 	(paper "A4")
+	(title_block
+		(title "FOME Open Source Wideband O2 Module")
+		(date "2026-03-22")
+		(rev "C")
+		(company "FOME / Happy Cactus Garage")
+		(comment 1 "github.com/mck1117/wideband")
+	)
 	(text "Un_sense = 2.7 * (Un - Vm)"
 		(exclude_from_sim no)

Commit message: update LED PNs
Parts:
- D2: LCSC C72043 -> C12624
- D3: LCSC C72041 -> C2288
Changed lines of the file:
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@@
 			)
 		)
-		(property "LCSC" "C72041"
+		(property "LCSC" "C2288"
 			(at 260.35 117.475 0)
 			(effects
@@
 			)
 		)
-		(property "LCSC" "C72043"
+		(property "LCSC" "C12624"
 			(at 260.35 108.585 0)
 			(effects
